Commit message: g1 backpack

File: source/whole_body_tracking/whole_body_tracking/assets/unitree_description/urdf/g1_23dof_backpack/main_with_backpack.urdf (robot description, URDF)
Before this commit: robot g1_23dof_rev_1_0, 32 links, 31 joints
Links:
- link thor_backpack_link: geometry collision mesh filename=meshes/backpack_link.STL; visual mesh filename=meshes/backpack_link.STL

Commit message: Use box collision for backpack to avoid mesh collision issues

File: source/whole_body_tracking/whole_body_tracking/assets/unitree_description/urdf/g1_23dof_backpack/main_with_backpack.urdf (robot description, URDF)
Before this commit: robot g1_23dof_rev_1_0, 32 links, 31 joints
Links:
- link thor_backpack_link: geometry collision box size=0.19 0.09 0.25; visual mesh filename=meshes/backpack_link.STL

Commit message: g1 backpack

File: source/whole_body_tracking/whole_body_tracking/assets/unitree_description/urdf/g1_23dof_backpack/main_with_backpack.urdf (robot description, URDF)
Before this commit: robot g1_23dof_rev_1_0, 32 links, 31 joints
Links:
- link thor_backpack_link: mass 1.9 -> None; geometry visual mesh filename=meshes/backpack_link.STL
- link torso_link: mass 6.78 -> 8.680000

Commit message: g1 backpack

File: source/whole_body_tracking/whole_body_tracking/assets/unitree_description/urdf/g1_23dof_backpack/main_with_backpack.urdf (robot description, URDF)
Before this commit: robot g1_23dof_rev_1_0, 32 links, 31 joints
Links:
- link thor_backpack_link: mass None -> 1.9; geometry collision box size=0.19 0.09 0.25; visual mesh filename=meshes/backpack_link.STL
- link torso_link: mass 8.680000 -> 6.78

Commit message: sync update

File: source/whole_body_tracking/whole_body_tracking/assets/unitree_description/urdf/g1_23dof_backpack/main_with_backpack.urdf (robot description, URDF)
Before this commit: robot g1_23dof_rev_1_0, 32 links, 31 joints
Links:
- link thor_backpack_link: geometry collision box size=0.092719 0.192405 0.246378; visual mesh filename=meshes/backpack_link.STL

Commit message: sync update

File: source/whole_body_tracking/whole_body_tracking/assets/unitree_description/urdf/g1_23dof_backpack/main_with_backpack.urdf (robot description, URDF)
Before this commit: robot g1_23dof_rev_1_0, 32 links, 31 joints
Links:
- link thor_backpack_link: mass 1.9 -> 0.8
